File: SIM808.sch (EAGLE design)
At the start: 0 parts

Commit message: SIM808 circuitry design
Parts:
- added C1, C2: 10uF, rcl:C-USC0805
- added C3: 100uF, rcl:C-USC0805
- added C4: 33pF, rcl:C-USC0805
- added C5: 100PF, rcl:C-USC0805
- added CN1: (no value), adafruit:USBMINIB
- added D1: BAT60J, diode:BAT60J
- added D2: SMF05C, SMF05C:SMF05C
- added J1: U.FL-R-SMT(01), U.FL-R-SMT_01_:U.FL-R-SMT(01)
- added LED1, LED2: (no value), led:LEDSML0805
- added R1: 470ohm, rcl:R-US_R0805
- added R2: 1K, rcl:R-US_R0805
- added R3: 10K, rcl:R-US_R0805
- added U$1: MCP73811T-420I/OT, MCP73811T-420I_OT:MCP73811T-420I/OT
- added U1: (no value), adafruit:GSM_SIM808_LITERAL
- added U2: SN74ABT125PW, SN74ABT125PW:SN74ABT125PW
- added X1: SMA-142-0701-801/806, con-coax:SMA-142-0701-801/806
- added X2: 5036_006_201_862, con-kyocera-elco:5036_006_201_862
Connections:
- new net +5V: C1.1, CN1.VBUS, LED1.A, U$1.VDD
- new net 1.8V: D2.C1, U1.SIM_VDD, X2.C1
- new net 2.8V: R3.1, U1.VDD_EXT(2.8VOUT)
- new net GND: C1.2, C2.2, C3.2, C4.2, C5.2, CN1.GND, D1.A, D2.A, J1.GND, R2.1, U$1.CE, U$1.VSS, U1.GND@1, U1.GND@10, U1.GND@11, U1.GND@12, U1.GND@13, U1.GND@14, U1.GND@15, U1.GND@2, U1.GND@3, U1.GND@4, U1.GND@5, U1.GND@6, U1.GND@7, U1.GND@9, X1.2, X2.C5
- new net GSM_RST: U1.RESET
- new net GSM_RXD: U1.RXD
- new net GSM_TXD: U1.TXD
- new net N$1: LED2.A, R1.2, U$1.PROG
- new net N$2: LED2.C, R2.2
- new net N$3: LED1.C, R1.1
- new net N$4: C2.1, U1.VRTC
- new net N$5: U1.GSM_RF_IN, X1.1
- new net N$6: J1.SIG, U1.GPS_RF_IN
- new net N$8: R3.2, U1.RTS
- new net NETSTAT: U1.NETLIGHT
- new net PWRKEY: U1.PWRKEY
- new net PWRSTAT: U1.STATUS
- new net RING: U1.RI
- new net SIM_CLK: D2.C3, U1.SIM_CLK, X2.C3
- new net SIM_DATA: D2.C2, U1.SIM_DATA, X2.C7
- new net SIM_RST: D2.C4, U1.SIM_RST, X2.C2
- new net VBAT: C3.1, C4.1, C5.1, D1.C, U$1.VBAT, U1.VBAT@1, U1.VBAT@2, U1.VBAT@3
